File: voltage_reg/voltage_reg.kicad_sch (KiCad schematic)
At the start: 7 parts, among them J1 USB_B_Micro, J2 Screw_Terminal_01x02, U1 AMS1117CD-3.3

Commit message: started to work on the pcb and poured some traces for 5v and 3v3
Parts:
- added C5: 22u, Capacitor_SMD:CP_Elec_6.3x7.7, symbol Device:C_Polarized_Small
- J1: footprint Connector_USB:USB_Micro-B_Amphenol_10118194_Horizontal -> Connector_USB:USB_Micro-B_Molex_47346-0001
Connections:
- net +3.3V: now also C5.1
- net GND: now also C5.2
Changed lines of the file:
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@@
 	(paper "A4")
+	(junction
+		(at 135.89 59.69)
+		(diameter 0)
+		(color 0 0 0 0)
+	)
 	(junction
 		(at 124.46 59.69)
@@
 	)
 	(junction
+		(at 135.89 77.47)
+		(diameter 0)
+		(color 0 0 0 0)
+	)
+	(junction
 		(at 80.01 59.69)
 		(diameter 0)
@@
 	(wire
 		(pts
-			(xy 143.51 59.69) (xy 124.46 59.69)
+			(xy 143.51 59.69) (xy 135.89 59.69)
 		)
 		(stroke
@@
 	(wire
 		(pts
+			(xy 135.89 59.69) (xy 124.46 59.69)
+		)
+		(stroke
+			(width 0)
+			(type default)
+		)
+	)
+	(wire
+		(pts
 			(xy 143.51 68.58) (xy 143.51 77.47)
 		)
@@
 	(wire
 		(pts
-			(xy 143.51 77.47) (xy 124.46 77.47)
+			(xy 143.51 77.47) (xy 135.89 77.47)
 		)
 		(stroke
@@
 	(wire
 		(pts
+			(xy 135.89 71.12) (xy 135.89 77.47)
+		)
+		(stroke
+			(width 0)
+			(type default)
+		)
+	)
+	(wire
+		(pts
 			(xy 124.46 77.47) (xy 107.95 77.47)
 		)
@@
 		(pts
 			(xy 69.85 54.61) (xy 69.85 59.69)
+		)
+		(stroke
+			(width 0)
+			(type default)
+		)
+	)
+	(wire
+		(pts
+			(xy 135.89 59.69) (xy 135.89 66.04)
+		)
+		(stroke
+			(width 0)
+			(type default)
+		)
+	)
+	(wire
+		(pts
+			(xy 135.89 77.47) (xy 124.46 77.47)
 		)
 		(stroke
@@
 	)
 	(symbol
+		(lib_id "Device:C_Polarized_Small")
+		(at 135.89 68.58 0)
+		(unit 1)
+		(exclude_from_sim no)
+		(in_bom yes)
+		(on_board yes)
+		(dnp no)
+		(fields_autoplaced yes)
+		(property "Reference" "C5"
+			(at 138.43 66.7638 0)
+			(effects
+				(font
+					(size 1.27 1.27)
+				)
+				(justify left)
+			)
+		)
+		(property "Value" "22u"
+			(at 138.43 69.3038 0)
+			(effects
+				(font
+					(size 1.27 1.27)
+				)
+				(justify left)
+			)
+		)
+		(property "Footprint" "Capacitor_SMD:CP_Elec_6.3x7.7"
+			(at 135.89 68.58 0)
+			(effects
+				(font
+					(size 1.27 1.27)
+				)
+				(hide yes)
+			)
+		)
+		(property "Datasheet" "~"
+			(at 135.89 68.58 0)
+			(effects
+				(font
+					(size 1.27 1.27)
+				)
+				(hide yes)
+			)
+		)
+		(property "Description" "Polarized capacitor, small symbol"
+			(at 135.89 68.58 0)
+			(effects
+				(font
+					(size 1.27 1.27)
+				)
+				(hide yes)
+			)
+		)
+		(property "part number" ""
+			(at 135.89 68.58 0)
+			(effects
+				(font
+					(size 1.27 1.27)
+				)
+				(hide yes)
+			)
+		)
+		(pin "1"
+		)
+		(pin "2"
+		)
+		(instances
+			(project "voltage_reg"
+				(path "/14871852-16ee-44e7-a0af-8a8c35c49ac5"
+					(reference "C5")
+					(unit 1)
+				)
+			)
+		)
+	)
+	(symbol
 		(lib_id "Device:C_Small")
 		(at 80.01 73.66 0)
@@
 			)
 		)
-		(property "Footprint" "Connector_USB:USB_Micro-B_Amphenol_10118194_Horizontal"
+		(property "Footprint" "Connector_USB:USB_Micro-B_Molex_47346-0001"
 			(at 54.61 66.04 0)
 			(effects
